Commit message: Adding Chevy Bolt features

File: src/mirvehicle_description/urdf/bulldogbolt/properties.urdf.xacro (robot description, xacro)
@@ -9,9 +9,11 @@
 <xacro:property name="wheelbase" value="2.6"/>
 <xacro:property name="track_width" value="1.501"/>
-<xacro:property name="car_height" value="1.594"/>
+<!-- TODO: fix the car_height -->
+<xacro:property name="car_height" value="1.4478"/> <!--1.594"/-->
 <xacro:property name="car_width" value="1.765"/>
 <xacro:property name="car_length" value="4.166"/>
-<xacro:property name="base_height" value="1.0639"/>
-<xacro:property name="base_mass" value="1625"/>
+<!-- TODO: fix the base_mass with its inertia -->
+<xacro:property name="base_height" value="1.04"/>
+<xacro:property name="base_mass" value="2050"/> <!--1625"/-->
 <xacro:property name="base_mass_ixx" value="63"/>
 <xacro:property name="base_mass_iyy" value="1048"/>
@@ -22,5 +24,6 @@
 <xacro:property name="tire_length" value="0.215"/>
 <xacro:property name="tire_diameter" value="0.6468"/>
-<xacro:property name="tire_radius" value="${tire_diameter/2}"/>
+<xacro:property name="tire_radius" value="0.356"/>
+<!-- TODO: fix the tire mass with its inertia -->
 <xacro:property name="tire_mass" value="40"/>
 <xacro:property name="tire_mass_ixx" value="54"/>
@@ -31,8 +34,13 @@
 </xacro:property>
 <xacro:property name="tire_origin_2">
-    <origin xyz="0 0 0" rpy="0 0 ${PI/2}"/>
+    <origin xyz="-0.3065 -0.765 1.372" rpy="0 0 ${-PI/2}"/>
 </xacro:property>
 <xacro:property name="tire_origin_3">
-    <origin xyz="0 0 0" rpy="0 0 ${-PI/2}"/>
+    <origin xyz="0.3065 0.765 1.372" rpy="0 0 ${PI/2}"/>
+</xacro:property>
+<xacro:property name="wheel_geometry">
+    <geometry>
+        <mesh filename="package://mirvehicle_description/meshes/$(arg robot_name)/wheel.dae" scale="0.0383 0.0383 0.0383"/>
+    </geometry>
 </xacro:property>
 <xacro:property name="dist_to_bumper" value="2.1"/>

File: src/mirvehicle_description/urdf/bulldogbolt/structure.urdf.xacro (robot description, xacro)
@@ -65,8 +65,5 @@
     <visual>
         <xacro:insert_block name="tire_origin_2"/>
-        <geometry>
-            <mesh filename="package://mirvehicle_description/meshes/$(arg robot_name)/wheel.dae"/>
-            <scale xyz="1.2 1 1"/>
-        </geometry>
+        <xacro:insert_block name="wheel_geometry"/>
     </visual>
     <inertial>
@@ -100,8 +97,5 @@
     <visual>
         <xacro:insert_block name="tire_origin_3"/>
-        <geometry>
-            <mesh filename="package://mirvehicle_description/meshes/$(arg robot_name)/wheel.dae"/>
-            <scale xyz="1.2 1 1"/>
-        </geometry>
+        <xacro:insert_block name="wheel_geometry"/>
     </visual>
     <inertial>
@@ -136,8 +130,5 @@
     <visual>
         <xacro:insert_block name="tire_origin_2"/>
-        <geometry>
-            <mesh filename="package://mirvehicle_description/meshes/$(arg robot_name)/wheel.dae"/>
-            <scale xyz="1.2 1 1"/>
-        </geometry>
+        <xacro:insert_block name="wheel_geometry"/>
      </visual>
     <inertial>
@@ -168,8 +159,5 @@
     <visual>
         <xacro:insert_block name="tire_origin_3"/>
-        <geometry>
-            <mesh filename="package://mirvehicle_description/meshes/$(arg robot_name)/wheel.dae"/>
-            <scale xyz="1.2 1 1"/>
-        </geometry>
+        <xacro:insert_block name="wheel_geometry"/>
     </visual>
     <inertial>

Commit message: Adding Chevy Bolt's features

File: src/mirvehicle_description/urdf/bulldogbolt/properties.urdf.xacro (robot description, xacro)
@@ -7,4 +7,44 @@
 <xacro:property name="PI" value="3.1415926835897931"/>
 <!--  <xacro:property name="base_height" value="0"/> -->
+<<<<<<< HEAD
+<xacro:property name="wheelbase" value="2.6"/>
+<xacro:property name="track_width" value="1.501"/>
+<!-- TODO: fix the car_height -->
+<xacro:property name="car_height" value="1.4478"/> <!--1.594"/-->
+<xacro:property name="car_width" value="1.765"/>
+<xacro:property name="car_length" value="4.166"/>
+<!-- TODO: fix the base_mass with its inertia -->
+<xacro:property name="base_height" value="1.04"/>
+<xacro:property name="base_mass" value="2050"/> <!--1625"/-->
+<xacro:property name="base_mass_ixx" value="63"/>
+<xacro:property name="base_mass_iyy" value="1048"/>
+<xacro:property name="base_mass_izz" value="1111"/>
+<xacro:property name="base_mass_ixz" value="-31"/>
+<xacro:property name="tire_x" value="${wheelbase/2}"/>
+<xacro:property name="tire_y" value="${track_width/2}"/>
+<xacro:property name="tire_length" value="0.215"/>
+<xacro:property name="tire_diameter" value="0.6468"/>
+<xacro:property name="tire_radius" value="0.356"/>
+<!-- TODO: fix the tire mass with its inertia -->
+<xacro:property name="tire_mass" value="40"/>
+<xacro:property name="tire_mass_ixx" value="54"/>
+<xacro:property name="tire_mass_iyy" value="56"/>
+<xacro:property name="tire_mass_izz" value="104"/>
+<xacro:property name="tire_origin">
+    <origin xyz="0 0 0" rpy="${PI/2} 0 0"/>
+</xacro:property>
+<xacro:property name="tire_origin_2">
+    <origin xyz="-0.3065 -0.765 1.372" rpy="0 0 ${-PI/2}"/>
+</xacro:property>
+<xacro:property name="tire_origin_3">
+    <origin xyz="0.3065 0.765 1.372" rpy="0 0 ${PI/2}"/>
+</xacro:property>
+<xacro:property name="wheel_geometry">
+    <geometry>
+        <mesh filename="package://mirvehicle_description/meshes/$(arg robot_name)/wheel.dae" scale="0.0383 0.0383 0.0383"/>
+    </geometry>
+</xacro:property>
+<xacro:property name="dist_to_bumper" value="2.1"/>
+=======
 <xacro:property name="base_height" value="1.1159"/>
 <xacro:property name="base_mass" value="1562"/>
@@ -24,8 +64,13 @@
 <xacro:property name="car_height" value="1.6"/>
 <xacro:property name="car_to_bumper" value="2.085"/>
+>>>>>>> 392b662d9e2527d674f22fc6910ae1a39eb32f01
 <xacro:property name="front_bumper_height" value="${car_height/2}"/>
 <xacro:property name="sensor_box" value="0.25"/>
-<xacro:property name="sensor_box2" value="0.31"/>
 <xacro:property name="camera_box" value="0.1"/>
+<<<<<<< HEAD
+<xacro:property name="steer_length" value="0.01"/>
+<xacro:property name="steer_radius" value="0.1"/>
+<xacro:property name="steer_angle_limit" value="0.6"/>
+=======
 <xacro:property name="tyre_height" value="-0.696"/>
 <xacro:property name="str_length" value="0.01"/>
@@ -33,10 +78,14 @@
 <xacro:property name="str_angle" value="0.6"/>
 <xacro:property name="car_width" value="1.3"/>
+>>>>>>> 392b662d9e2527d674f22fc6910ae1a39eb32f01
 <xacro:property name="front_laser_points" value="$(arg front_laser_points)"/>
 <xacro:property name="velodyne_points" value="$(arg velodyne_points)"/>
 <xacro:property name="camera_right" value="$(arg camera_right)"/>
 <xacro:property name="camera_left" value="$(arg camera_left)"/>
+<<<<<<< HEAD
+=======
 <xacro:property name="tyre_origin">
     <origin xyz="0 0 0" rpy="${PI/2} 0 0"/>
 </xacro:property>
+>>>>>>> 392b662d9e2527d674f22fc6910ae1a39eb32f01
 </robot>

File: src/mirvehicle_description/urdf/bulldogbolt/sensors.urdf.xacro (robot description, xacro)
@@ -33,5 +33,9 @@
 <!-- ********************************************************************** -->
 <joint name="camera_left_joint" type="fixed">
+<<<<<<< HEAD
+    <origin xyz="-0.75 ${track_width/2-0.12} ${0.525 + camera_box/2 + 1.25}" rpy="0 0 ${PI/2}"/>
+=======
     <origin xyz="-0.75 0.5 ${0.595 + camera_box/2 + 1.25}" rpy="0 0 ${PI/2}"/>
+>>>>>>> 392b662d9e2527d674f22fc6910ae1a39eb32f01
     <axis xyz="0 0 1"/>
     <parent link="base_link"/>
@@ -61,5 +65,9 @@
 <!-- ********************************************************************** -->
 <joint name="camera_right_joint" type="fixed">
+<<<<<<< HEAD
+    <origin xyz="-0.75 -${track_width/2-0.12} ${0.525 + camera_box/2 + 1.25}" rpy="0 0 -${PI/2}"/>
+=======
     <origin xyz="-0.75 -0.5 ${0.595 + camera_box/2 + 1.25}" rpy="0 0 -${PI/2}"/>
+>>>>>>> 392b662d9e2527d674f22fc6910ae1a39eb32f01
     <axis xyz="0 0 1"/>
     <parent link="base_link"/>
@@ -89,5 +97,9 @@
 <!-- ********************************************************************** -->
 <joint name="camera_joint" type="fixed">
+<<<<<<< HEAD
+    <origin xyz="0 0 ${0.725 + sensor_box/2 + 1.15}" rpy="0 0 0"/>
+=======
     <origin xyz="0 0 ${0.595+ sensor_box/2 + 1.25}" rpy="0 0 0"/>
+>>>>>>> 392b662d9e2527d674f22fc6910ae1a39eb32f01
     <axis xyz="0 0 1"/>
     <parent link="base_link"/>
@@ -145,5 +157,5 @@
 <!-- ********************************************************************** -->
 <joint name="front_laser_joint" type="fixed">
-    <origin xyz="${car_to_bumper} 0 ${front_bumper_height + sensor_box/2 + 0.01}" rpy="0 0 0"/>
+    <origin xyz="${dist_to_bumper} 0 ${front_bumper_height + sensor_box/2 + 0.01}" rpy="0 0 0"/>
     <axis xyz="0 0 1"/>
     <parent link="base_link"/>

File: src/mirvehicle_description/urdf/bulldogbolt/structure.urdf.xacro (robot description, xacro)
@@ -11,5 +11,5 @@
         <origin xyz="0 0 ${base_height}" rpy="0 0 0"/>
         <geometry>
-            <box size="2.62 ${car_width} ${car_height}"/>
+            <box size="${car_length} ${car_width} ${car_height}"/>
         </geometry>
     </collision>
@@ -50,5 +50,9 @@
     <parent link="base_link"/>
     <child link="back_left_wheel_link"/>
+<<<<<<< HEAD
+    <origin xyz="${-tire_x} ${tire_y} ${tire_diameter}" rpy="0 0 0"/>
+=======
     <origin xyz="${-tyre_x} ${tyre_y} 0.608" rpy="0 0 0"/>
+>>>>>>> 392b662d9e2527d674f22fc6910ae1a39eb32f01
     <axis xyz="0 1 0"/>
     <dynamics damping="0.1"/>
@@ -58,22 +62,27 @@
 <link name="back_left_wheel_link">
     <collision>
-        <xacro:insert_block name="tyre_origin"/>
-        <geometry>
-            <cylinder length="${tyre_length}" radius="${tyre_radius}"/>
-        </geometry>
-    </collision>
-    <visual>
+        <xacro:insert_block name="tire_origin"/>
+        <geometry>
+            <cylinder length="${tire_length}" radius="${tire_radius}"/>
+        </geometry>
+    </collision>
+    <visual>
+<<<<<<< HEAD
+        <xacro:insert_block name="tire_origin_2"/>
+        <xacro:insert_block name="wheel_geometry"/>
+=======
         <origin xyz="-0.3065 -0.765 1.372" rpy="0 0 ${-PI/2}"/>
         <geometry>
             <mesh filename="package://mirvehicle_description/meshes/$(arg robot_name)/wheel.dae" scale="0.0383 0.0383 0.0383"/>
         </geometry>
-    </visual>
-    <inertial>
-        <origin xyz="0 0 0" rpy="0 0 0"/>
-        <mass value="${tyre_mass}"/>
-        <inertia
-            ixx="${tyre_mass_ixx}"  ixy="0.000000"  ixz="0.000000"
-            iyy="${tyre_mass_iyy}"  iyz="0.000000"
-            izz="${tyre_mass_izz}"/>
+>>>>>>> 392b662d9e2527d674f22fc6910ae1a39eb32f01
+    </visual>
+    <inertial>
+        <origin xyz="0 0 0" rpy="0 0 0"/>
+        <mass value="${tire_mass}"/>
+        <inertia
+            ixx="${tire_mass_ixx}"  ixy="0.000000"  ixz="0.000000"
+            iyy="${tire_mass_iyy}"  iyz="0.000000"
+            izz="${tire_mass_izz}"/>
     </inertial>
 </link>
@@ -84,5 +93,9 @@
     <parent link="base_link"/>
     <child link="back_right_wheel_link"/>
+<<<<<<< HEAD
+    <origin xyz="${-tire_x} ${-tire_y} ${tire_diameter}" rpy="0 0 0"/>
+=======
     <origin xyz="${-tyre_x} ${-tyre_y} 0.608" rpy="0 0 0"/>
+>>>>>>> 392b662d9e2527d674f22fc6910ae1a39eb32f01
     <axis xyz="0 1 0"/>
     <dynamics damping="0.1"/>
@@ -92,22 +105,27 @@
 <link name="back_right_wheel_link">
     <collision>
-        <xacro:insert_block name="tyre_origin"/>
-        <geometry>
-            <cylinder length="${tyre_length}" radius="${tyre_radius}"/>
-        </geometry>
-    </collision>
-    <visual>
+        <xacro:insert_block name="tire_origin"/>
+        <geometry>
+            <cylinder length="${tire_length}" radius="${tire_radius}"/>
+        </geometry>
+    </collision>
+    <visual>
+<<<<<<< HEAD
+        <xacro:insert_block name="tire_origin_3"/>
+        <xacro:insert_block name="wheel_geometry"/>
+=======
         <origin xyz="0.3065 0.765 1.372" rpy="0 0 ${PI/2}"/>
         <geometry>
             <mesh filename="package://mirvehicle_description/meshes/$(arg robot_name)/wheel.dae" scale="0.0383 0.0383 0.0383"/>
         </geometry>
-    </visual>
-    <inertial>
-        <origin xyz="0 0 0" rpy="0 0 0"/>
-        <mass value="${tyre_mass}"/>
-        <inertia
-            ixx="${tyre_mass_ixx}"  ixy="0.000000"  ixz="0.000000"
-            iyy="${tyre_mass_iyy}"  iyz="0.000000"
-            izz="${tyre_mass_izz}"/>
+>>>>>>> 392b662d9e2527d674f22fc6910ae1a39eb32f01
+    </visual>
+    <inertial>
+        <origin xyz="0 0 0" rpy="0 0 0"/>
+        <mass value="${tire_mass}"/>
+        <inertia
+            ixx="${tire_mass_ixx}"  ixy="0.000000"  ixz="0.000000"
+            iyy="${tire_mass_iyy}"  iyz="0.000000"
+            izz="${tire_mass_izz}"/>
     </inertial>
 </link>
@@ -118,5 +136,5 @@
     <parent link="front_left_steering_link"/>
     <child link="front_left_wheel_link"/>
-    <origin xyz="0 ${str_length/2 + tyre_length/2} 0" rpy="0 0 0"/>
+    <origin xyz="0 ${steer_length/2 + tire_length/2} 0" rpy="0 0 0"/>
     <axis xyz="0 1 0"/>
     <dynamics damping="0.1"/>
@@ -129,20 +147,25 @@
         <origin xyz="0 0 0" rpy="${PI/2} 0 0"/>
         <geometry>
-             <cylinder length="${tyre_length}" radius="${tyre_radius}"/>
-        </geometry>
-    </collision>
-    <visual>
+             <cylinder length="${tire_length}" radius="${tire_radius}"/>
+        </geometry>
+    </collision>
+    <visual>
+<<<<<<< HEAD
+        <xacro:insert_block name="tire_origin_2"/>
+        <xacro:insert_block name="wheel_geometry"/>
+=======
         <origin xyz="-0.3065 -0.765 1.372" rpy="0 0 ${-PI/2}"/>
         <geometry>
             <mesh filename="package://mirvehicle_description/meshes/$(arg robot_name)/wheel.dae" scale="0.0383 0.0383 0.0383"/>
         </geometry>
+>>>>>>> 392b662d9e2527d674f22fc6910ae1a39eb32f01
      </visual>
     <inertial>
         <origin xyz="0 0 0" rpy="0 0 0"/>
-        <mass value="${tyre_mass}"/>
-        <inertia
-            ixx="${tyre_mass_ixx}"  ixy="0.000000"  ixz="0.000000"
-            iyy="${tyre_mass_iyy}"  iyz="0.000000"
-            izz="${tyre_mass_izz}"/>
+        <mass value="${tire_mass}"/>
+        <inertia
+            ixx="${tire_mass_ixx}"  ixy="0.000000"  ixz="0.000000"
+            iyy="${tire_mass_iyy}"  iyz="0.000000"
+            izz="${tire_mass_izz}"/>
     </inertial>
 </link>
@@ -153,27 +176,32 @@
     <parent link="front_right_steering_link"/>
     <child link="front_right_wheel_link"/>
-    <origin xyz="0 ${-str_length/2 - tyre_length/2} 0" rpy="0 0 0"/>
+    <origin xyz="0 ${-steer_length/2 - tire_length/2} 0" rpy="0 0 0"/>
     <axis xyz="0 1 0"/>
 </joint>
 <link name="front_right_wheel_link">
     <collision>
-        <xacro:insert_block name="tyre_origin"/>
-        <geometry>
-            <cylinder length="${tyre_length}" radius="${tyre_radius}"/>
-        </geometry>
-    </collision>
-    <visual>
+        <xacro:insert_block name="tire_origin"/>
+        <geometry>
+            <cylinder length="${tire_length}" radius="${tire_radius}"/>
+        </geometry>
+    </collision>
+    <visual>
+<<<<<<< HEAD
+        <xacro:insert_block name="tire_origin_3"/>
+        <xacro:insert_block name="wheel_geometry"/>
+=======
         <origin xyz="0.3065 0.765 1.372" rpy="0 0 ${PI/2}"/>
         <geometry>
             <mesh filename="package://mirvehicle_description/meshes/$(arg robot_name)/wheel.dae" scale="0.0383 0.0383 0.0383"/>
         </geometry>
-    </visual>
-    <inertial>
-        <origin xyz="0 0 0" rpy="0 0 0"/>
-        <mass value="${tyre_mass}"/>
+>>>>>>> 392b662d9e2527d674f22fc6910ae1a39eb32f01
+    </visual>
+    <inertial>
+        <origin xyz="0 0 0" rpy="0 0 0"/>
+        <mass value="${tire_mass}"/>
     <inertia
-        ixx="${tyre_mass_ixx}"  ixy="0.000000"  ixz="0.000000"
-        iyy="${tyre_mass_iyy}"  iyz="0.000000"
-        izz="${tyre_mass_izz}"/>
+        ixx="${tire_mass_ixx}"  ixy="0.000000"  ixz="0.000000"
+        iyy="${tire_mass_iyy}"  iyz="0.000000"
+        izz="${tire_mass_izz}"/>
     </inertial>
 </link>
@@ -184,20 +212,24 @@
     <parent link="base_link"/>
     <child link="front_left_steering_link"/>
+<<<<<<< HEAD
+    <origin xyz="${tire_x} ${tire_y - (tire_length+steer_length)/2} ${tire_diameter}" rpy="0 0 0"/>
+=======
     <origin xyz="${tyre_x} ${car_width/2 + str_length/2} 0.608" rpy="0 0 0"/>
+>>>>>>> 392b662d9e2527d674f22fc6910ae1a39eb32f01
     <axis xyz="0 0 1"/>
-    <limit effort="1000.0" lower="${-str_angle}" upper="${str_angle}" velocity="0.5"/>
+    <limit effort="1000.0" lower="${-steer_angle_limit}" upper="${steer_angle_limit}" velocity="0.5"/>
 </joint>
 <link name="front_left_steering_link">
     <!-- ?? parent link="base_link"/ -->
     <collision>
-        <xacro:insert_block name="tyre_origin"/>
-        <geometry>
-            <cylinder length="${str_length}" radius="${str_radius}"/>
-        </geometry>
-    </collision>
-    <visual>
-        <xacro:insert_block name="tyre_origin"/>
-        <geometry>
-            <cylinder length="${str_length}" radius="${str_radius}"/>
+        <xacro:insert_block name="tire_origin"/>
+        <geometry>
+            <cylinder length="${steer_length}" radius="${steer_radius}"/>
+        </geometry>
+    </collision>
+    <visual>
+        <xacro:insert_block name="tire_origin"/>
+        <geometry>
+            <cylinder length="${steer_length}" radius="${steer_radius}"/>
         </geometry>
     </visual>
@@ -217,19 +249,23 @@
     <parent link="base_link"/>
     <child link="front_right_steering_link"/>
+<<<<<<< HEAD
+    <origin xyz="${tire_x} ${-tire_y + (tire_length+steer_length)/2} ${tire_diameter}" rpy="0 0 0"/>
+=======
     <origin xyz="${tyre_x} ${-car_width/2 - str_length/2} 0.608" rpy="0 0 0"/>
+>>>>>>> 392b662d9e2527d674f22fc6910ae1a39eb32f01
     <axis xyz="0 0 1"/>
-    <limit effort="1000.0" lower="${-str_angle}" upper="${str_angle}" velocity="0.5"/>
+    <limit effort="1000.0" lower="${-steer_angle_limit}" upper="${steer_angle_limit}" velocity="0.5"/>
 </joint>
 <link name="front_right_steering_link">
     <collision>
-        <xacro:insert_block name="tyre_origin"/>
-        <geometry>
-            <cylinder length="${str_length}" radius="${str_radius}"/>
-        </geometry>
-    </collision>
-    <visual>
-        <xacro:insert_block name="tyre_origin"/>
-        <geometry>
-            <cylinder length="${str_length}" radius="${str_radius}"/>
+        <xacro:insert_block name="tire_origin"/>
+        <geometry>
+            <cylinder length="${steer_length}" radius="${steer_radius}"/>
+        </geometry>
+    </collision>
+    <visual>
+        <xacro:insert_block name="tire_origin"/>
+        <geometry>
+            <cylinder length="${steer_length}" radius="${steer_radius}"/>
         </geometry>
     </visual>
