Commit message: Milestone 1: It works!

File: src/mirvehicle_description/urdf/bulldogbolt/sensors.urdf.xacro (robot description, xacro)
@@ -24,135 +24,148 @@
     <xacro:include filename="$(find mirvehicle_description)/urdf/mirvehicle_left_camera_gazebo.urdf.xacro"/>
 </xacro:if>
-<!-- ====================================================================== -->
-<!-- Cameras-->
+!-- ********************************************************************** -->
+<!-- ********************************************************************** -->
+<!-- Sensors -->
+<!-- ********************************************************************** -->
+<!-- ********************************************************************** -->
+<!-- ********************************************************************** -->
+<!-- Left Camera-->
+<!-- ********************************************************************** -->
+<joint name="camera_left_joint" type="fixed">
+    <origin xyz="-0.75 ${car_width/2} ${0.725 + camera_box/2 + 1.25}" rpy="0 0 ${PI/2}"/>
+    <axis xyz="0 0 1"/>
+    <parent link="base_link"/>
+    <child link="camera_left_link"/>
+</joint>
+<link name="camera_left_link">
+    <collision>
+        <origin xyz="0 0 0" rpy="0 0 0"/>
+        <geometry>
+            <box size="${camera_box} ${camera_box} ${camera_box}"/>
+        </geometry>
+    </collision>
+    <visual>
+        <origin xyz="0 0 0" rpy="0 0 0"/>
+        <geometry>
+            <box size="${camera_box} ${camera_box} ${camera_box}"/>
+        </geometry>
+    </visual>
+    <inertial>
+        <mass value="1e-5" />
+        <origin xyz="0 0 0" rpy="0 0 0"/>
+        <inertia ixx="1e-6" ixy="0" ixz="0" iyy="1e-6" iyz="0" izz="1e-6" />
+    </inertial>
+</link>
+<!-- ********************************************************************** -->
+<!-- Right Camera-->
+<!-- ********************************************************************** -->
 <joint name="camera_right_joint" type="fixed">
-<origin xyz="-0.75 -${car_width/2} ${0.725 + camera_box/2 + 1.25}" rpy="0 0 -${PI/2}"/>
-	<axis xyz="0 0 1"/>
-	<parent link="base_link"/>
-	<child link="camera_right_link"/>
+    <origin xyz="-0.75 -${car_width/2} ${0.725 + camera_box/2 + 1.25}" rpy="0 0 -${PI/2}"/>
+    <axis xyz="0 0 1"/>
+    <parent link="base_link"/>
+    <child link="camera_right_link"/>
 </joint>
 <link name="camera_right_link">
-	<collision>
-	  <origin xyz="0 0 0" rpy="0 0 0"/>
-	  <geometry>
-	   <box size="${camera_box} ${camera_box} ${camera_box}"/>
-	  </geometry>
-	</collision>
-	<visual>
-	  <origin xyz="0 0 0" rpy="0 0 0"/>
-	  <geometry>
-	  <box size="${camera_box} ${camera_box} ${camera_box}"
-/>
-          </geometry>
-	</visual>
+    <collision>
+        <origin xyz="0 0 0" rpy="0 0 0"/>
+        <geometry>
+            <box size="${camera_box} ${camera_box} ${camera_box}"/>
+        </geometry>
+    </collision>
+    <visual>
+        <origin xyz="0 0 0" rpy="0 0 0"/>
+        <geometry>
+            <box size="${camera_box} ${camera_box} ${camera_box}"/>
+        </geometry>
+    </visual>
     <inertial>
-      <mass value="1e-5" />
-      <origin xyz="0 0 0" rpy="0 0 0"/>
-      <inertia ixx="1e-6" ixy="0" ixz="0" iyy="1e-6" iyz="0" izz="1e-6" />
+        <mass value="1e-5" />
+        <origin xyz="0 0 0" rpy="0 0 0"/>
+        <inertia ixx="1e-6" ixy="0" ixz="0" iyy="1e-6" iyz="0" izz="1e-6" />
     </inertial>
 </link>
-<joint name="camera_left_joint" type="fixed">
-<origin xyz="-0.75 ${car_width/2} ${0.725 + camera_box/2 + 1.25}" rpy="0 0 ${PI/2}"/>
-	<axis xyz="0 0 1"/>
-	<parent link="base_link"/>
-	<child link="camera_left_link"/>
+<!-- ********************************************************************** -->
+<!-- Camera Joint -->
+<!-- ********************************************************************** -->
+<joint name="camera_joint" type="fixed">
+    <origin xyz="0 0 ${0.725 + sensor_box/2 + 1.25}" rpy="0 0 0"/>
+    <axis xyz="0 0 1"/>
+    <parent link="base_link"/>
+    <child link="camera_link"/>
 </joint>
-<link name="camera_left_link">
-	<collision>
-	  <origin xyz="0 0 0" rpy="0 0 0"/>
-	  <geometry>
-	   <box size="${camera_box} ${camera_box} ${camera_box}"/>
-	  </geometry>
-	</collision>
-	<visual>
-	  <origin xyz="0 0 0" rpy="0 0 0"/>
-	  <geometry>
-	  <box size="${camera_box} ${camera_box} ${camera_box}"
-/>
-          </geometry>
-	</visual>
+<link name="camera_link">
+    <collision>
+        <origin xyz="0 0 0" rpy="0 0 0"/>
+        <geometry>
+            <box size="${sensor_box} ${sensor_box} ${sensor_box}"/>
+        </geometry>
+    </collision>
+    <visual>
+        <origin xyz="0 0 0" rpy="0 0 0"/>
+        <geometry>
+            <box size="${sensor_box} ${sensor_box} ${sensor_box}"/>
+        </geometry>
+    </visual>
     <inertial>
-      <mass value="1e-5" />
-      <origin xyz="0 0 0" rpy="0 0 0"/>
-      <inertia ixx="1e-6" ixy="0" ixz="0" iyy="1e-6" iyz="0" izz="1e-6" />
+        <mass value="1e-5" />
+        <origin xyz="0 0 0" rpy="0 0 0"/>
+        <inertia ixx="1e-6" ixy="0" ixz="0" iyy="1e-6" iyz="0" izz="1e-6" />
     </inertial>
 </link>
-<joint name="camera_joint" type="fixed">
-<origin xyz="0 0 ${0.725 + sensor_box/2 + 1.25}" rpy="0 0 0"/>
-	<axis xyz="0 0 1"/>
-	<parent link="base_link"/>
-	<child link="camera_link"/>
+<!-- ********************************************************************** -->
+<!--Velodyne LIDAR-->
+<!-- ********************************************************************** -->
+<joint name="velodyne_joint" type="fixed">
+    <origin xyz="0 0 ${sensor_box/2 + 0.01}" rpy="0 0 0"/>
+    <axis xyz="0 0 1"/>
+    <parent link="camera_link"/>
+    <child link="velodyne_link"/>
 </joint>
-<link name="camera_link">
-	<collision>
-	  <origin xyz="0 0 0" rpy="0 0 0"/>
-	  <geometry>
-	   <box size="${sensor_box} ${sensor_box} ${sensor_box}"/>
-	  </geometry>
-	</collision>
-	<visual>
-	  <origin xyz="0 0 0" rpy="0 0 0"/>
-	  <geometry>
-	  <box size="${sensor_box} ${sensor_box} ${sensor_box}"
-/>
-          </geometry>
-	</visual>
+<link name="velodyne_link">
+    <collision>
+        <origin xyz="0 0 0" rpy="0 0 0"/>
+        <geometry>
+            <box size="${sensor_box} ${sensor_box} ${sensor_box}"/>
+        </geometry>
+    </collision>
+    <visual>
+        <origin xyz="0 0 0" rpy="0 0 0"/>
+        <geometry>
+            <box size="${sensor_box} ${sensor_box} ${sensor_box}"/>
+        </geometry>
+    </visual>
     <inertial>
-      <mass value="1e-5" />
-      <origin xyz="0 0 0" rpy="0 0 0"/>
-      <inertia ixx="1e-6" ixy="0" ixz="0" iyy="1e-6" iyz="0" izz="1e-6" />
+        <mass value="1e-5" />
+        <origin xyz="0 0 0" rpy="0 0 0"/>
+        <inertia ixx="1e-6" ixy="0" ixz="0" iyy="1e-6" iyz="0" izz="1e-6" />
     </inertial>
 </link>
-<!-- ====================================================================== -->
-<!--Velodyne LIDAR-->
-<joint name="velodyne_joint" type="fixed">
-	<origin xyz="0 0 ${sensor_box/2 + 0.01}" rpy="0 0 0"/>
-	<axis xyz="0 0 1"/>
-	<parent link="camera_link"/>
-	<child link="velodyne_link"/>
-</joint>
-<link name="velodyne_link">
-        <collision>
-          <origin xyz="0 0 0" rpy="0 0 0"/>
-          <geometry>
-           <box size="${sensor_box} ${sensor_box} ${sensor_box}"/>
-          </geometry>
-        </collision>
-        <visual>
-          <origin xyz="0 0 0" rpy="0 0 0"/>
-          <geometry>
-           <box size="${sensor_box} ${sensor_box} ${sensor_box}"/>
-          </geometry>
-        </visual>
-    <inertial>
-      <mass value="1e-5" />
-      <origin xyz="0 0 0" rpy="0 0 0"/>
-      <inertia ixx="1e-6" ixy="0" ixz="0" iyy="1e-6" iyz="0" izz="1e-6" />
-    </inertial>
-</link>
+<!-- ********************************************************************** -->
+<!-- SICKLIDAR-->
+<!-- ********************************************************************** -->
 <joint name="front_laser_joint" type="fixed">
-	<origin xyz="${car_to_bumper} 0 ${front_bumper_height + sensor_box/2 + 0.01}" rpy="0 0 0"/>
-	<axis xyz="0 0 1"/>
-	<parent link="base_link"/>
-	<child link="front_laser_link"/>
+    <origin xyz="${car_to_bumper} 0 ${front_bumper_height + sensor_box/2 + 0.01}" rpy="0 0 0"/>
+    <axis xyz="0 0 1"/>
+    <parent link="base_link"/>
+    <child link="front_laser_link"/>
 </joint>
 <link name="front_laser_link">
-     <parent link="front_laser_joint"/>
-        <collision>
-          <origin xyz="0 0 0" rpy="0 0.0 0"/>
-          <geometry>
-           <box size="${sensor_box} ${sensor_box} ${sensor_box}"/>
-          </geometry>
-        </collision>
-        <visual>
-          <origin xyz="0 0 0" rpy="0 0 0"/>
-          <geometry>
-           <box size="${sensor_box} ${sensor_box} ${sensor_box}"/>
-          </geometry>
-        </visual>
+    <parent link="front_laser_joint"/>
+    <collision>
+        <origin xyz="0 0 0" rpy="0 0.0 0"/>
+        <geometry>
+            <box size="${sensor_box} ${sensor_box} ${sensor_box}"/>
+        </geometry>
+    </collision>
+    <visual>
+        <origin xyz="0 0 0" rpy="0 0 0"/>
+        <geometry>
+            <box size="${sensor_box} ${sensor_box} ${sensor_box}"/>
+        </geometry>
+    </visual>
     <inertial>
-      <mass value="1e-5" />
-      <origin xyz="0 0 0" rpy="0 0 0"/>
-      <inertia ixx="1e-6" ixy="0" ixz="0" iyy="1e-6" iyz="0" izz="1e-6" />
+        <mass value="1e-5" />
+        <origin xyz="0 0 0" rpy="0 0 0"/>
+        <inertia ixx="1e-6" ixy="0" ixz="0" iyy="1e-6" iyz="0" izz="1e-6" />
     </inertial>
 </link>

File: src/mirvehicle_description/urdf/mirvehicle_gazebo.urdf.xacro (robot description, xacro)
@@ -32,8 +32,8 @@
 # Author: Jaerock Kwon
 # ============================================================================
-# 12/1/2017: Change the package name to mirvehicle
-# 12/6/2017: Change kp in front_left/right_wheel_link to the same as
-#            back_left/right_wheel_link
-#
+# 12/01/2017: Change the package name to mirvehicle
+# 12/06/2017: Change kp in front_left/right_wheel_link to the same as
+#             back_left/right_wheel_link
+# 12/11/2017: Add proper joint names for RWD/FWD. Bulldogbolt is FWD.
 # ============================================================================
 -->
@@ -58,16 +58,16 @@
     <mu1>10000</mu1>
     <mu2>10000</mu2>
-    <kp>10000000</kp>
+    <kp>1000000</kp>
     <kd>1</kd>
     <minDepth>0.01</minDepth>
-    <maxVel>10.0</maxVel>
+    <maxVel>100.0</maxVel>
 </gazebo>
 <gazebo reference="front_left_wheel_link">
     <mu1>10000</mu1>
     <mu2>10000</mu2>
-    <kp>10000000</kp>
+    <kp>1000000</kp>
     <kd>1</kd>
     <minDepth>0.01</minDepth>
-    <maxVel>10.0</maxVel>
+    <maxVel>100.0</maxVel>
 </gazebo>
 <gazebo reference="front_right_steering_link">
@@ -95,5 +95,8 @@
 <gazebo>
     <plugin filename="libgazebo_ros_joint_state_publisher.so" name="joint_state_publisher">
-        <jointName>back_left_wheel_joint, back_right_wheel_joint, front_left_steering_joint, front_right_steering_joint, front_right_wheel_joint, front_left_wheel_joint</jointName>
+      <!-- RWD -->
+      <!-- jointName>back_left_wheel_joint, back_right_wheel_joint, front_left_steering_joint, front_right_steering_joint, front_right_wheel_joint, front_left_wheel_joint</jointName -->
+      <!-- FWD -->
+      <jointName>front_left_wheel_joint, front_right_wheel_joint, front_left_steering_joint, front_right_steering_joint, front_right_wheel_joint, front_left_wheel_joint</jointName>
         <updateRate>50.0</updateRate>
         <robotNamespace>/$(arg robot_name)</robotNamespace>

Commit message: First commit

File: src/mirvehicle_description/urdf/bulldogbolt/sensors.urdf.xacro (robot description, xacro)
@@ -33,5 +33,5 @@
 <!-- ********************************************************************** -->
 <joint name="camera_left_joint" type="fixed">
-    <origin xyz="-0.75 0.5 ${0.595 + camera_box/2 + 1.25}" rpy="0 0 ${PI/2}"/>
+    <origin xyz="0.58 0 ${0.595 + camera_box/2 + 1.05}" rpy="0 0 0"/>
     <axis xyz="0 0 1"/>
     <parent link="base_link"/>

File: src/mirvehicle_description/urdf/bulldogbolt/structure.urdf.xacro (robot description, xacro)
@@ -155,4 +155,7 @@
     <origin xyz="0 ${-str_length/2 - tyre_length/2} 0" rpy="0 0 0"/>
     <axis xyz="0 1 0"/>
+    <dynamics damping="0.1"/>
+    <limit effort="10000" velocity="100" />
+    <joint_properties damping="0.0" friction="0.0" />
 </joint>
 <link name="front_right_wheel_link">
@@ -256,8 +259,8 @@
     <!-- FWD -->
     <joint name="front_left_wheel_joint">
-        <hardwareInterface>hardware_interface/VelocityJointInterface</hardwareInterface>
+        <hardwareInterface>VelocityJointInterface</hardwareInterface>
     </joint>
     <actuator name="motor1">
-        <hardwareInterface>hardware_interface/VelocityJointInterface</hardwareInterface>
+        <hardwareInterface>VelocityJointInterface</hardwareInterface>
         <mechanicalReduction>1</mechanicalReduction>
     </actuator>
@@ -269,8 +272,8 @@
     <!-- FWD -->
     <joint name="front_right_wheel_joint">
-        <hardwareInterface>hardware_interface/VelocityJointInterface</hardwareInterface>
+        <hardwareInterface>VelocityJointInterface</hardwareInterface>
     </joint>
     <actuator name="motor2">
-        <hardwareInterface>hardware_interface/VelocityJointInterface</hardwareInterface>
+        <hardwareInterface>VelocityJointInterface</hardwareInterface>
         <mechanicalReduction>1</mechanicalReduction>
     </actuator>
@@ -279,8 +282,8 @@
     <type>transmission_interface/SimpleTransmission</type>
         <joint name="front_left_steering_joint">
-        <hardwareInterface>hardware_interface/PositionJointInterface</hardwareInterface>
+        <hardwareInterface>PositionJointInterface</hardwareInterface>
     </joint>
     <actuator name="eps_left">
-        <hardwareInterface>hardware_interface/PositionJointInterface</hardwareInterface>
+        <hardwareInterface>PositionJointInterface</hardwareInterface>
         <mechanicalReduction>1</mechanicalReduction>
     </actuator>
@@ -289,8 +292,8 @@
     <type>transmission_interface/SimpleTransmission</type>
         <joint name="front_right_steering_joint">
-        <hardwareInterface>hardware_interface/PositionJointInterface</hardwareInterface>
+        <hardwareInterface>PositionJointInterface</hardwareInterface>
     </joint>
     <actuator name="eps_right">
-        <hardwareInterface>hardware_interface/PositionJointInterface</hardwareInterface>
+        <hardwareInterface>PositionJointInterface</hardwareInterface>
         <mechanicalReduction>1</mechanicalReduction>
     </actuator>
